Commit message: update1

File: slam_project/urdf/udacity_bot.xacro (robot description, xacro)
@@ -139,5 +139,5 @@
     <joint_properties damping="1.0" friction="1.0"/>
   </joint>
-<link name ="camera">
+<link name ="camera_link">
 <origin xyz="0 0 0" rpy="0 0 0"/>
 <collision>
@@ -160,5 +160,5 @@
 <joint type="fixed" name="camera_joint">
 <orign xyz="0.2 0 0" rpy="0 0 0"/>
-<child link="camera"/>
+<child link="camera_link"/>
 <parent link="chassis"/>
 </joint>

Commit message: Updates as 9/2
removed the references for udacity_bot

File: slam_project/urdf/udacity_bot.xacro (robot description, xacro)
@@ -1,4 +1,4 @@
 <?xml version='1.0'?>
-<robot name="udacity_bot" xmlns:xacro="http://www.ros.org/wiki/xacro">
+<robot name="slam_project" xmlns:xacro="http://www.ros.org/wiki/xacro">
 <material name="blue">
     <color rgba="0 0 0.8 1"/>
@@ -7,5 +7,5 @@
     <color rgba="0 1 0 1"/>
   </material>
-<xacro:include filename="$(find udacity_bot)/urdf/udacity_bot.gazebo" />
+<xacro:include filename="$(find slam_project)/urdf/udacity_bot.gazebo" />
   <link name="robot_footprint"></link>
   <joint name="robot_footprint_joint" type="fixed">
@@ -173,5 +173,5 @@
 <visual>
 	<geometry>
-	 <mesh filename="package://udacity_bot/meshes/hokuyo.dae"/>
+	 <mesh filename="package://slam_project/meshes/hokuyo.dae"/>
 	</geometry>
 </visual>

Commit message: status as 9_15
1)Now the rgb frame is showing in the tf
2) pointcloud is showing but in upward direction .. to fix

File: slam_project/urdf/udacity_bot.xacro (robot description, xacro)
@@ -147,4 +147,5 @@
 </geometry>
 </collision>
+<!--
 <visual>
 <origin xyz="0.2 0 0" rpy="0 0 0"/>
@@ -152,4 +153,10 @@
 <box size="0.05 0.05 0.05"/>
 </geometry>
+</visual>
+-->
+<visual name="visual">
+        <geometry>
+         <mesh filename="package://slam_project/meshes/kinect.dae"/>
+        </geometry>
 </visual>
 <inertial>
@@ -163,4 +170,10 @@
 <parent link="chassis"/>
 </joint>
+<joint type="fixed" name="rgb_camera_joint">
+<orign xyz="0.2 0 0" rpy="0 0 0"/>
+<parent link="camera_link"/>
+<child link="camera_rgbd_frame"/>
+</joint>
+<link name="camera_rgbd_frame"/>
 <link name="hokuyo">
 <origin xyz="0 0 0" rpy="0 0 0"/>

Commit message: re-committing after removal of big files

File: slam_project/urdf/udacity_bot.xacro (robot description, xacro)
@@ -139,5 +139,5 @@
     <joint_properties damping="1.0" friction="1.0"/>
   </joint>
-<link name ="camera_link">
+<link name ="camera">
 <origin xyz="0 0 0" rpy="0 0 0"/>
 <collision>
@@ -167,13 +167,14 @@
 <joint type="fixed" name="camera_joint">
 <orign xyz="0.2 0 0" rpy="0 0 0"/>
-<child link="camera_link"/>
+<child link="camera"/>
 <parent link="chassis"/>
 </joint>
-<joint type="fixed" name="rgb_camera_joint">
+<joint type="fixed" name="camera_optical_joint">
 <orign xyz="0 0 0" rpy="${-pi/2} 0 ${-pi/2}"/>
-<parent link="camera_link"/>
-<child link="camera_rgbd_frame"/>
+<parent link="camera"/>
+<child link="camera_link_optical"/>
 </joint>
-<link name="camera_rgbd_frame"/>
+<!-- <link name="camera_rgbd_frame"/> -->
+<link name="camera_link_optical"/>
 <link name="hokuyo">
 <origin xyz="0 0 0" rpy="0 0 0"/>

Commit message: finally ... got the good picture

File: slam_project/urdf/udacity_bot.xacro (robot description, xacro)
@@ -166,10 +166,10 @@
 </link>
 <joint type="fixed" name="camera_joint">
-<orign xyz="0.2 0 0" rpy="0 0 0"/>
+<origin xyz="0.2 0 0" rpy="0 0 0"/>
 <child link="camera"/>
 <parent link="chassis"/>
 </joint>
 <joint type="fixed" name="camera_optical_joint">
-<orign xyz="0 0 0" rpy="${-pi/2} 0 ${-pi/2}"/>
+<origin xyz="0 0 0" rpy="${-pi/2} 0 ${-pi/2}"/>
 <parent link="camera"/>
 <child link="camera_link_optical"/>
